File: Codigo fuente/Circuito mallas.brd (EAGLE design)
At the start: 56.8 x 53.3 mm, 7 parts, among them P1 18V, P2 5V

Commit message: Add files via upload
Parts:
- added Meter1, Meter2, Meter3: (no value), AUTODESK_CIRCUITS_BREADBOARD:DC-POWER
Connections:
- removed net N$2 (its old number): P1.2, R1.1
- removed net N$3 (its old number): P1.1, P2.1, R2.1, R5.1
- new net N$1: Meter1.+, P1.2
- new net N$4: Meter2.-, R3.1, R5.2
- new net N$6: Meter3.+, P2.1
- new net N$7: Meter1.-, R1.1
- new net N$8: Meter2.+, R4.1
- net N$5: now also Meter3.-, P1.1, R2.1, R5.1; no longer R3.1, R4.1, R5.2
Changed lines of the file:
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@@
 </autorouter>
 <elements>
-<element value="820‎Ω" name="R1" library="AUTODESK_CIRCUITS_BREADBOARD" package="0207/10" x="5" y="10.08"></element><element value="1k‎Ω" name="R2" library="AUTODESK_CIRCUITS_BREADBOARD" package="0207/10" x="5" y="22.78"></element><element value="390‎Ω" name="R3" library="AUTODESK_CIRCUITS_BREADBOARD" package="0207/10" x="5" y="35.480000000000004"></element><element value="1.2k‎Ω" name="R4" library="AUTODESK_CIRCUITS_BREADBOARD" package="0207/10" x="5" y="48.18"></element><element value="2.2k‎Ω" name="R5" library="AUTODESK_CIRCUITS_BREADBOARD" package="0207/10" x="5" y="60.879999999999995"></element><element value="18V" name="P1" library="AUTODESK_CIRCUITS_BREADBOARD" package="2P-2.54-65/35MIL" x="5" y="73.58"></element><element value="5V" name="P2" library="AUTODESK_CIRCUITS_BREADBOARD" package="2P-2.54-65/35MIL" x="5" y="86.28"></element></elements>
+<element value="820‎Ω" name="R1" library="AUTODESK_CIRCUITS_BREADBOARD" package="0207/10" x="5" y="10.08"></element><element value="1k‎Ω" name="R2" library="AUTODESK_CIRCUITS_BREADBOARD" package="0207/10" x="5" y="22.78"></element><element value="390‎Ω" name="R3" library="AUTODESK_CIRCUITS_BREADBOARD" package="0207/10" x="5" y="35.480000000000004"></element><element value="1.2k‎Ω" name="R4" library="AUTODESK_CIRCUITS_BREADBOARD" package="0207/10" x="5" y="48.18"></element><element value="2.2k‎Ω" name="R5" library="AUTODESK_CIRCUITS_BREADBOARD" package="0207/10" x="5" y="60.879999999999995"></element><element value="18V" name="P1" library="AUTODESK_CIRCUITS_BREADBOARD" package="2P-2.54-65/35MIL" x="5" y="73.58"></element><element value="5V" name="P2" library="AUTODESK_CIRCUITS_BREADBOARD" package="2P-2.54-65/35MIL" x="5" y="86.28"></element><element value="" name="Meter1" library="AUTODESK_CIRCUITS_BREADBOARD" package="DC-POWER" x="5" y="98.98"></element><element value="" name="Meter2" library="AUTODESK_CIRCUITS_BREADBOARD" package="DC-POWER" x="5" y="111.68"></element><element value="" name="Meter3" library="AUTODESK_CIRCUITS_BREADBOARD" package="DC-POWER" x="5" y="124.38000000000001"></element></elements>
 <signals>
-<signal name="N$1"><contactref element="R1" pad="2"></contactref><contactref element="R2" pad="2"></contactref><wire x1="10.08" y1="10.08" x2="10.08" y2="22.78" width="0" layer="19" extent="1-1"></wire><contactref element="R4" pad="2"></contactref><wire x1="10.08" y1="22.78" x2="10.08" y2="48.18" width="0" layer="19" extent="1-1"></wire></signal><signal name="N$2"><contactref element="R1" pad="1"></contactref><contactref element="P1" pad="2"></contactref><wire x1="-0.08000000000000007" y1="10.08" x2="5" y2="72.31" width="0" layer="19" extent="1-1"></wire></signal><signal name="N$3"><contactref element="R5" pad="1"></contactref><contactref element="P2" pad="1"></contactref><wire x1="-0.08000000000000007" y1="60.879999999999995" x2="5" y2="87.55" width="0" layer="19" extent="1-1"></wire><contactref element="R2" pad="1"></contactref><wire x1="5" y1="87.55" x2="-0.08000000000000007" y2="22.78" width="0" layer="19" extent="1-1"></wire><contactref element="P1" pad="1"></contactref><wire x1="-0.08000000000000007" y1="22.78" x2="5" y2="74.85" width="0" layer="19" extent="1-1"></wire></signal><signal name="N$4"><contactref element="R3" pad="2"></contactref><contactref element="P2" pad="2"></contactref><wire x1="10.08" y1="35.480000000000004" x2="5" y2="85.01" width="0" layer="19" extent="1-1"></wire></signal><signal name="N$5"><contactref element="R4" pad="1"></contactref><contactref element="R5" pad="2"></contactref><wire x1="-0.08000000000000007" y1="48.18" x2="10.08" y2="60.879999999999995" width="0" layer="19" extent="1-1"></wire><contactref element="R3" pad="1"></contactref><wire x1="10.08" y1="60.879999999999995" x2="-0.08000000000000007" y2="35.480000000000004" width="0" layer="19" extent="1-1"></wire></signal></signals>
+<signal name="N$1"><contactref element="P1" pad="2"></contactref><contactref element="Meter1" pad="+"></contactref><wire x1="5" y1="72.31" x2="5" y2="101.52000000000001" width="0" layer="19" extent="1-1"></wire></signal><signal name="N$2"><contactref element="R1" pad="2"></contactref><contactref element="R2" pad="2"></contactref><wire x1="10.08" y1="10.08" x2="10.08" y2="22.78" width="0" layer="19" extent="1-1"></wire><contactref element="R4" pad="2"></contactref><wire x1="10.08" y1="22.78" x2="10.08" y2="48.18" width="0" layer="19" extent="1-1"></wire></signal><signal name="N$3"><contactref element="R3" pad="2"></contactref><contactref element="P2" pad="2"></contactref><wire x1="10.08" y1="35.480000000000004" x2="5" y2="85.01" width="0" layer="19" extent="1-1"></wire></signal><signal name="N$4"><contactref element="R3" pad="1"></contactref><contactref element="R5" pad="2"></contactref><wire x1="-0.08000000000000007" y1="35.480000000000004" x2="10.08" y2="60.879999999999995" width="0" layer="19" extent="1-1"></wire><contactref element="Meter2" pad="-"></contactref><wire x1="10.08" y1="60.879999999999995" x2="5" y2="109.14" width="0" layer="19" extent="1-1"></wire></signal><signal name="N$5"><contactref element="R5" pad="1"></contactref><contactref element="R2" pad="1"></contactref><wire x1="-0.08000000000000007" y1="60.879999999999995" x2="-0.08000000000000007" y2="22.78" width="0" layer="19" extent="1-1"></wire><contactref element="P1" pad="1"></contactref><wire x1="-0.08000000000000007" y1="22.78" x2="5" y2="74.85" width="0" layer="19" extent="1-1"></wire><contactref element="Meter3" pad="-"></contactref><wire x1="5" y1="74.85" x2="5" y2="121.84" width="0" layer="19" extent="1-1"></wire></signal><signal name="N$6"><contactref element="P2" pad="1"></contactref><contactref element="Meter3" pad="+"></contactref><wire x1="5" y1="87.55" x2="5" y2="126.92000000000002" width="0" layer="19" extent="1-1"></wire></signal><signal name="N$7"><contactref element="R1" pad="1"></contactref><contactref element="Meter1" pad="-"></contactref><wire x1="-0.08000000000000007" y1="10.08" x2="5" y2="96.44" width="0" layer="19" extent="1-1"></wire></signal><signal name="N$8"><contactref element="R4" pad="1"></contactref><contactref element="Meter2" pad="+"></contactref><wire x1="-0.08000000000000007" y1="48.18" x2="5" y2="114.22000000000001" width="0" layer="19" extent="1-1"></wire></signal></signals>
 </board>
 </drawing>
